File: PCB/Tetris/Tetris.kicad_sch (KiCad schematic)
At the start: 9 parts, among them J1 Power, J2 PWM, J3 Analog, J4 PWM, J5 Analog, J6 Communication, J7 Digital, M1 RGBMatrix, M2 RGBMatrix

Commit message: something happened
Parts:
- added R1, R2, R3, R4, R5, R6, R7, R8: 110, symbol Device:R
- M1, M2: footprint (none) -> RGBMatrix:RGBMatrix
Connections:
- net at M1.17 (P_1): now also R1.2
- net at M1.18 (P_2): now also R2.2
- net at M1.19 (P_3): now also R3.2
- net at M1.20 (P_4): now also R4.2
- net at M1.29 (P_5): now also R5.2
- net at M1.30 (P_6): now also R6.2
- net at M1.31 (P_7): now also R7.2
- net at M1.32 (P_8): now also R8.2
Other:
- moved on the sheet: M1, M2
Changed lines of the file:
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@@
     )
   )
-  (symbol (lib_id "RGBMatrix:RGBMatrix") (at 105.918 38.735 0) (unit 1)
-    (in_bom yes) (on_board yes) (dnp no) (fields_autoplaced)
-    (property "Reference" "M2" (at 127.635 24.1553 0)
+  (symbol (lib_id "Device:R") (at 113.03 76.2 0) (unit 1)
+    (in_bom yes) (on_board yes) (dnp no) (fields_autoplaced)
+    (property "Reference" "R7" (at 115.57 75.565 0)
+      (effects (font (size 1.27 1.27)) (justify left))
+    )
+    (property "Value" "110" (at 115.57 78.105 0)
+      (effects (font (size 1.27 1.27)) (justify left))
+    )
+    (property "Footprint" "" (at 111.252 76.2 90)
+      (effects (font (size 1.27 1.27)) hide)
+    )
+    (property "Datasheet" "~" (at 113.03 76.2 0)
+      (effects (font (size 1.27 1.27)) hide)
+    )
+    (pin "1")
+    (pin "2")
+    (instances
+      (project "Tetris"
+        (path "/e63e39d7-6ac0-4ffd-8aa3-1841a4541b55"
+          (reference "R7") (unit 1)
+        )
+      )
+    )
+  )
+  (symbol (lib_id "RGBMatrix:RGBMatrix") (at 119.38 41.91 0) (unit 1)
+    (in_bom yes) (on_board yes) (dnp no) (fields_autoplaced)
+    (property "Reference" "M2" (at 141.097 27.3303 0)
       (effects (font (size 1.27 1.27)))
     )
-    (property "Value" "RGBMatrix" (at 127.635 26.6953 0)
+    (property "Value" "RGBMatrix" (at 141.097 29.8703 0)
       (effects (font (size 1.27 1.27)))
     )
-    (property "Footprint" "" (at 105.918 34.925 0)
-      (effects (font (size 1.27 1.27)) hide)
-    )
-    (property "Datasheet" "" (at 105.918 34.925 0)
+    (property "Footprint" "RGBMatrix:RGBMatrix" (at 119.38 38.1 0)
+      (effects (font (size 1.27 1.27)) hide)
+    )
+    (property "Datasheet" "" (at 119.38 38.1 0)
       (effects (font (size 1.27 1.27)) hide)
     )
@@
     )
   )
+  (symbol (lib_id "Device:R") (at 118.11 76.2 0) (unit 1)
+    (in_bom yes) (on_board yes) (dnp no) (fields_autoplaced)
+    (property "Reference" "R5" (at 120.65 75.565 0)
+      (effects (font (size 1.27 1.27)) (justify left))
+    )
+    (property "Value" "110" (at 120.65 78.105 0)
+      (effects (font (size 1.27 1.27)) (justify left))
+    )
+    (property "Footprint" "" (at 116.332 76.2 90)
+      (effects (font (size 1.27 1.27)) hide)
+    )
+    (property "Datasheet" "~" (at 118.11 76.2 0)
+      (effects (font (size 1.27 1.27)) hide)
+    )
+    (pin "1")
+    (pin "2")
+    (instances
+      (project "Tetris"
+        (path "/e63e39d7-6ac0-4ffd-8aa3-1841a4541b55"
+          (reference "R5") (unit 1)
+        )
+      )
+    )
+  )
+  (symbol (lib_id "Device:R") (at 115.57 76.2 0) (unit 1)
+    (in_bom yes) (on_board yes) (dnp no) (fields_autoplaced)
+    (property "Reference" "R6" (at 118.11 75.565 0)
+      (effects (font (size 1.27 1.27)) (justify left))
+    )
+    (property "Value" "110" (at 118.11 78.105 0)
+      (effects (font (size 1.27 1.27)) (justify left))
+    )
+    (property "Footprint" "" (at 113.792 76.2 90)
+      (effects (font (size 1.27 1.27)) hide)
+    )
+    (property "Datasheet" "~" (at 115.57 76.2 0)
+      (effects (font (size 1.27 1.27)) hide)
+    )
+    (pin "1")
+    (pin "2")
+    (instances
+      (project "Tetris"
+        (path "/e63e39d7-6ac0-4ffd-8aa3-1841a4541b55"
+          (reference "R6") (unit 1)
+        )
+      )
+    )
+  )
   (symbol (lib_id "power:VCC") (at 26.67 26.67 0) (unit 1)
     (in_bom yes) (on_board yes) (dnp no)
@@
     )
   )
-  (symbol (lib_id "RGBMatrix:RGBMatrix") (at 106.299 75.565 0) (unit 1)
-    (in_bom yes) (on_board yes) (dnp no) (fields_autoplaced)
-    (property "Reference" "M1" (at 127.635 60.9853 0)
+  (symbol (lib_id "Device:R") (at 128.27 76.2 0) (unit 1)
+    (in_bom yes) (on_board yes) (dnp no) (fields_autoplaced)
+    (property "Reference" "R1" (at 130.81 75.565 0)
+      (effects (font (size 1.27 1.27)) (justify left))
+    )
+    (property "Value" "110" (at 130.81 78.105 0)
+      (effects (font (size 1.27 1.27)) (justify left))
+    )
+    (property "Footprint" "" (at 126.492 76.2 90)
+      (effects (font (size 1.27 1.27)) hide)
+    )
+    (property "Datasheet" "~" (at 128.27 76.2 0)
+      (effects (font (size 1.27 1.27)) hide)
+    )
+    (pin "1")
+    (pin "2")
+    (instances
+      (project "Tetris"
+        (path "/e63e39d7-6ac0-4ffd-8aa3-1841a4541b55"
+          (reference "R1") (unit 1)
+        )
+      )
+    )
+  )
+  (symbol (lib_id "Device:R") (at 120.65 76.2 0) (unit 1)
+    (in_bom yes) (on_board yes) (dnp no) (fields_autoplaced)
+    (property "Reference" "R4" (at 123.19 75.565 0)
+      (effects (font (size 1.27 1.27)) (justify left))
+    )
+    (property "Value" "110" (at 123.19 78.105 0)
+      (effects (font (size 1.27 1.27)) (justify left))
+    )
+    (property "Footprint" "" (at 118.872 76.2 90)
+      (effects (font (size 1.27 1.27)) hide)
+    )
+    (property "Datasheet" "~" (at 120.65 76.2 0)
+      (effects (font (size 1.27 1.27)) hide)
+    )
+    (pin "1")
+    (pin "2")
+    (instances
+      (project "Tetris"
+        (path "/e63e39d7-6ac0-4ffd-8aa3-1841a4541b55"
+          (reference "R4") (unit 1)
+        )
+      )
+    )
+  )
+  (symbol (lib_id "Device:R") (at 123.19 76.2 0) (unit 1)
+    (in_bom yes) (on_board yes) (dnp no) (fields_autoplaced)
+    (property "Reference" "R3" (at 125.73 75.565 0)
+      (effects (font (size 1.27 1.27)) (justify left))
+    )
+    (property "Value" "110" (at 125.73 78.105 0)
+      (effects (font (size 1.27 1.27)) (justify left))
+    )
+    (property "Footprint" "" (at 121.412 76.2 90)
+      (effects (font (size 1.27 1.27)) hide)
+    )
+    (property "Datasheet" "~" (at 123.19 76.2 0)
+      (effects (font (size 1.27 1.27)) hide)
+    )
+    (pin "1")
+    (pin "2")
+    (instances
+      (project "Tetris"
+        (path "/e63e39d7-6ac0-4ffd-8aa3-1841a4541b55"
+          (reference "R3") (unit 1)
+        )
+      )
+    )
+  )
+  (symbol (lib_id "Device:R") (at 125.73 76.2 0) (unit 1)
+    (in_bom yes) (on_board yes) (dnp no) (fields_autoplaced)
+    (property "Reference" "R2" (at 128.27 75.565 0)
+      (effects (font (size 1.27 1.27)) (justify left))
+    )
+    (property "Value" "110" (at 128.27 78.105 0)
+      (effects (font (size 1.27 1.27)) (justify left))
+    )
+    (property "Footprint" "" (at 123.952 76.2 90)
+      (effects (font (size 1.27 1.27)) hide)
+    )
+    (property "Datasheet" "~" (at 125.73 76.2 0)
+      (effects (font (size 1.27 1.27)) hide)
+    )
+    (pin "1")
+    (pin "2")
+    (instances
+      (project "Tetris"
+        (path "/e63e39d7-6ac0-4ffd-8aa3-1841a4541b55"
+          (reference "R2") (unit 1)
+        )
+      )
+    )
+  )
+  (symbol (lib_id "RGBMatrix:RGBMatrix") (at 119.38 96.52 0) (unit 1)
+    (in_bom yes) (on_board yes) (dnp no) (fields_autoplaced)
+    (property "Reference" "M1" (at 140.716 81.9403 0)
       (effects (font (size 1.27 1.27)))
     )
-    (property "Value" "RGBMatrix" (at 127.635 63.5253 0)
+    (property "Value" "RGBMatrix" (at 140.716 84.4803 0)
       (effects (font (size 1.27 1.27)))
     )
-    (property "Footprint" "" (at 106.299 71.755 0)
-      (effects (font (size 1.27 1.27)) hide)
-    )
-    (property "Datasheet" "" (at 106.299 71.755 0)
+    (property "Footprint" "RGBMatrix:RGBMatrix" (at 119.38 92.71 0)
+      (effects (font (size 1.27 1.27)) hide)
+    )
+    (property "Datasheet" "" (at 119.38 92.71 0)
       (effects (font (size 1.27 1.27)) hide)
     )
@@
         )
       )
+    )
+  )
+  (symbol (lib_id "Device:R") (at 110.49 76.2 0) (unit 1)
+    (in_bom yes) (on_board yes) (dnp no) (fields_autoplaced)
+    (property "Reference" "R8" (at 113.03 75.565 0)
+      (effects (font (size 1.27 1.27)) (justify left))
+    )
+    (property "Value" "110" (at 113.03 78.105 0)
+      (effects (font (size 1.27 1.27)) (justify left))
+    )
+    (property "Footprint" "" (at 108.712 76.2 90)
+      (effects (font (size 1.27 1.27)) hide)
+    )
+    (property "Datasheet" "~" (at 110.49 76.2 0)
+      (effects (font (size 1.27 1.27)) hide)
+    )
+    (pin "1")
+    (pin "2")
+    (instances
+      (project "Tetris"
+        (path "/e63e39d7-6ac0-4ffd-8aa3-1841a4541b55"
+          (reference "R8") (unit 1)
+        )
+      )

Commit message: Schematics and sync
Parts:
- removed J1: Power, Connector_PinSocket_2.54mm:PinSocket_1x08_P2.54mm_Vertical, symbol Connector_Generic:Conn_01x08
- removed M2: RGBMatrix, RGBMatrix:RGBMatrix, symbol RGBMatrix:RGBMatrix
- added BZ1, BZ2, BZ3, BZ4: Passive Buzzer, symbol Device:Buzzer
- added BZ5: Active Buzzer, symbol Device:Buzzer
- added DS1: WC1602A, Display:WC1602A, symbol Display_Character:WC1602A
- added RV1: R_Potentiometer_Trim, symbol Device:R_Potentiometer_Trim
- added RV3: R_Potentiometer, symbol Device:R_Potentiometer
- added SW1, SW2, SW3, SW4, SW5, SW6, SW7: SW_Push, symbol Switch:SW_Push
Connections:
- net 1: now reaches M1.1 (B_1)
- net 1: now also M1.10 (R_2), M1.11 (R_3), M1.12 (R_4), M1.13 (R_5), M1.14 (R_6), M1.15 (R_7), M1.16 (R_8), M1.2 (B_2), M1.21 (G_1), M1.22 (G_2), M1.23 (G_3), M1.24 (G_4), M1.25 (G_5), M1.26 (G_6), M1.27 (G_7), M1.28 (G_8), M1.3 (B_3), M1.4 (B_4), M1.5 (B_5), M1.6 (B_6), M1.7 (B_7), M1.8 (B_8), M1.9 (R_1)
- no-connect marks 1 -> 0
Other:
- note added: "Tetris Arudino Mega Shield"
- moved on the sheet: J2, J3, J4, J5, J6, J7, M1

Commit message: Sync change
Parts:
- removed DS1: WC1602A, Display:WC1602A, symbol Display_Character:WC1602A
- removed RV1: R_Potentiometer_Trim, symbol Device:R_Potentiometer_Trim
- removed RV3: R_Potentiometer, symbol Device:R_Potentiometer
- added M2: RGBMatrix, RGBMatrix:RGBMatrix, symbol RGBMatrix:RGBMatrix
- added R10, R11, R12, R13, R14, R15, R16, R9: 110, symbol Device:R
- added R17, R18, R19, R20, R21: 220, symbol Device:R
- BZ1, BZ2, BZ3, BZ4, BZ5: footprint (none) -> Buzzer_Beeper:MagneticBuzzer_PUI_AT-0927-TT-6-R
- SW1, SW2, SW3, SW4, SW5, SW6, SW7: footprint (none) -> Button_Switch_THT:SW_PUSH_6mm_H4.3mm
Connections:
- net 1: now also M2.1 (B_1), M2.10 (R_2), M2.11 (R_3), M2.12 (R_4), M2.13 (R_5), M2.14 (R_6), M2.15 (R_7), M2.16 (R_8), M2.2 (B_2), M2.21 (G_1), M2.22 (G_2), M2.23 (G_3), M2.24 (G_4), M2.25 (G_5), M2.26 (G_6), M2.27 (G_7), M2.28 (G_8), M2.3 (B_3), M2.4 (B_4), M2.5 (B_5), M2.6 (B_6), M2.7 (B_7), M2.8 (B_8), M2.9 (R_1)
- new net: M2.17 (P_1), R16.2
- new net: M2.31 (P_7), R10.2
- new net: M2.29 (P_5), R12.2
- new net: M2.18 (P_2), R15.2
- new net: M2.19 (P_3), R14.2
- new net: M2.20 (P_4), R13.2
- new net: M2.30 (P_6), R11.2
- new net: M2.32 (P_8), R9.2

Commit message: sync
Parts:
- removed BZ5: Active Buzzer, Buzzer_Beeper:MagneticBuzzer_PUI_AT-0927-TT-6-R, symbol Device:Buzzer
- added R22, R23, R24, R25, R26, R27: 110, Resistor_THT:R_Axial_DIN0207_L6.3mm_D2.5mm_P10.16mm_Horizontal, symbol Device:R
- BZ1, BZ2, BZ3, BZ4: footprint Buzzer_Beeper:MagneticBuzzer_PUI_AT-0927-TT-6-R -> Buzzer_Beeper:Buzzer_TDK_PS1240P02BT_D12.2mm_H6.5mm
- J2: footprint Connector_PinSocket_2.54mm:PinSocket_1x10_P2.54mm_Vertical -> Connector_PinHeader_2.54mm:PinHeader_1x10_P2.54mm_Vertical
- J4, J6: footprint Connector_PinSocket_2.54mm:PinSocket_1x08_P2.54mm_Vertical -> Connector_PinHeader_2.54mm:PinHeader_1x08_P2.54mm_Vertical
- R1, R2, R3, R4, R5, R6, R7, R8: footprint (none) -> Resistor_THT:R_Axial_DIN0207_L6.3mm_D2.5mm_P10.16mm_Horizontal
- R10, R11, R12, R9: value 110 -> 220; footprint (none) -> Resistor_THT:R_Axial_DIN0207_L6.3mm_D2.5mm_P10.16mm_Horizontal
- R13, R14, R15, R16: value 110 -> 10k; footprint (none) -> Resistor_THT:R_Axial_DIN0207_L6.3mm_D2.5mm_P10.16mm_Horizontal
- R17, R18, R19: value 220 -> 10k; footprint (none) -> Resistor_THT:R_Axial_DIN0207_L6.3mm_D2.5mm_P10.16mm_Horizontal
- R20, R21: value 220 -> 110; footprint (none) -> Resistor_THT:R_Axial_DIN0207_L6.3mm_D2.5mm_P10.16mm_Horizontal
Connections:
- net 1: no longer M1.10 (R_2), M1.11 (R_3), M1.12 (R_4), M1.13 (R_5), M1.14 (R_6), M1.15 (R_7), M1.16 (R_8), M1.2 (B_2), M1.21 (G_1), M1.22 (G_2), M1.23 (G_3), M1.24 (G_4), M1.25 (G_5), M1.26 (G_6), M1.27 (G_7), M1.28 (G_8), M1.3 (B_3), M1.4 (B_4), M1.5 (B_5), M1.6 (B_6), M1.7 (B_7), M1.8 (B_8), M1.9 (R_1), M2.10 (R_2), M2.11 (R_3), M2.12 (R_4), M2.13 (R_5), M2.14 (R_6), M2.15 (R_7), M2.16 (R_8), M2.2 (B_2), M2.21 (G_1), M2.22 (G_2), M2.23 (G_3), M2.24 (G_4), M2.25 (G_5), M2.26 (G_6), M2.27 (G_7), M2.28 (G_8), M2.3 (B_3), M2.4 (B_4), M2.5 (B_5), M2.6 (B_6), M2.7 (B_7), M2.8 (B_8), M2.9 (R_1)
- net 22: now also M1.22 (G_2), M2.22 (G_2)
- net 23: now also M1.23 (G_3), M2.23 (G_3)
- net 24: now also M1.24 (G_4), M2.24 (G_4)
- net 25: now also M1.25 (G_5), M2.25 (G_5)
- net 26: now also M1.26 (G_6), M2.26 (G_6)
- net 27: now also M1.27 (G_7), M2.27 (G_7)
- net 28: now also M1.28 (G_8), M2.28 (G_8)
- net 29: now also R5.1, R23.1
- net 30: now also R6.1, R22.1
- net 31: now also R21.1, R7.1
- net 32: now also R20.1, R8.1
- net at R16.2: no longer M2.17 (P_1)
- net at R10.2: no longer M2.31 (P_7)
- net at M2.29 (P_5): now also R23.2; no longer R12.2
- net at M2.18 (P_2): now also R26.2; no longer R15.2
- net at M2.19 (P_3): now also R25.2; no longer R14.2
- net at M2.20 (P_4): now also R24.2; no longer R13.2
- net at M2.30 (P_6): now also R22.2; no longer R11.2
- net at M2.32 (P_8): now also R20.2; no longer R9.2
- net 20: now reaches R4.1
- net 20: now also R24.1
- net 19: now reaches R3.1
- net 19: now also R25.1
- net 18: now reaches R2.1
- net 18: now also R26.1
- net 17: now reaches R1.1
- net 17: now also R27.1
- net at R21.2: now also M2.31 (P_7)
- new net: M2.17 (P_1), R27.2
- new net 10: M1.10 (R_2), M2.10 (R_2)
- new net 11: M1.11 (R_3), M2.11 (R_3)
- new net 12: M1.12 (R_4), M2.12 (R_4)
- new net 13: M1.13 (R_5), M2.13 (R_5)
- new net 14: M1.14 (R_6), M2.14 (R_6)
- new net 15: M1.15 (R_7), M2.15 (R_7)
- new net 16: M1.16 (R_8), M2.16 (R_8)
- new net 2: M1.2 (B_2), M2.2 (B_2)
- new net 21: M1.21 (G_1), M2.21 (G_1)
- new net 3: M1.3 (B_3), M2.3 (B_3)
- new net 4: M1.4 (B_4), M2.4 (B_4)
- new net 5: M1.5 (B_5), M2.5 (B_5)
- new net 6: M1.6 (B_6), M2.6 (B_6)
- new net 7: M1.7 (B_7), M2.7 (B_7)
- new net 8: M1.8 (B_8), M2.8 (B_8)
- new net 9: M1.9 (R_1), M2.9 (R_1)
Other:
- moved on the sheet: BZ1, BZ2, BZ3, BZ4, J2, J3, J4, J5, J6, J7, M1, R1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

Commit message: Making diabolical progress
Parts:
- removed R20, R21, R22, R23, R24, R25, R26, R27: 110, Resistor_THT:R_Axial_DIN0207_L6.3mm_D2.5mm_P10.16mm_Horizontal, symbol Device:R
- added R10, R11, R12, R13, R14, R15, R16, R9: 110, Resistor_THT:R_Axial_DIN0207_L6.3mm_D2.5mm_P10.16mm_Horizontal, symbol Device:R
- added U1: 74AHC595, Package_DIP:DIP-16_W7.62mm_Socket_LongPads, symbol 74xx:74AHC595
- J3, J5: footprint Connector_PinSocket_2.54mm:PinSocket_1x08_P2.54mm_Vertical -> Connector_PinHeader_2.54mm:PinHeader_1x08_P2.54mm_Vertical
- J7: footprint Connector_PinSocket_2.54mm:PinSocket_2x18_P2.54mm_Vertical -> Connector_PinHeader_2.54mm:PinHeader_2x18_P2.54mm_Vertical
- renumbered R13 to R17, R14 to R18, R15 to R19, R16 to R20, R17 to R21, R18 to R22, R19 to R23, R9 to R24, R10 to R25, R11 to R26, R12 to R27, R8 to R5, R7 to R6, R6 to R7, R5 to R8
Connections:
- net 17 is gone; now on net 28: R1.1
- net 18 is gone; now on net 26: R2.1
- net 19 is gone; now on net 24: R3.1
- net 20 is gone; now on net 22: R4.1
- net *10: now also BZ4.1 (-)
- net *11: now also BZ3.1 (-)
- net *12: now also BZ2.1 (-)
- net *13: now also BZ1.1 (-)
- net *2: now also M2.28 (G_8)
- net *3: now also M2.27 (G_7)
- net *4: now also M2.26 (G_6)
- net *5: now also M2.25 (G_5)
- net *6: now also M2.24 (G_4)
- net *7: now also M2.23 (G_3)
- net *8: now also M2.22 (G_2)
- net *9: now also M2.21 (G_1)
- net +5V: now also SW1.2, SW2.2, SW3.2, SW4.2, SW5.2, SW6.2, SW7.2
- net 22: now also R12.1; no longer M1.22 (G_2), M2.22 (G_2)
- net 23: now also R17.2, SW1.1; no longer M1.23 (G_3), M2.23 (G_3)
- net 24: now also R11.1; no longer M1.24 (G_4), M2.24 (G_4)
- net 25: now also R23.1, SW7.1; no longer M1.25 (G_5), M2.25 (G_5)
- net 26: now also R10.1; no longer M1.26 (G_6), M2.26 (G_6)
- net 27: now also R18.2, SW2.1; no longer M1.27 (G_7), M2.27 (G_7)
- net 28: now also R9.1; no longer M1.28 (G_8), M2.28 (G_8)
- net 29: no longer R8.1
- net 30: now also R8.2, R16.2; no longer R7.1
- net 31: now also R19.2, SW3.1; no longer R6.1
- net 32: now also R7.2, R15.2; no longer R5.1
- net 33: now also R21.2, SW5.1
- net 34: now also R6.2, R14.2
- net 36: now also R5.2, R13.2
- net 37: now also R22.1, SW6.1
- net 41: now also R20.2, SW4.1
- net 53: now also M1.1 (B_1)
- net A1: now also M1.2 (B_2)
- net A10: now also M1.11 (R_3)
- net A11: now also M1.12 (R_4)
- net A12: now also M1.13 (R_5)
- net A13: now also M1.14 (R_6)
- net A14: now also M1.15 (R_7)
- net A15: now also M1.16 (R_8)
- net A2: now also M1.3 (B_3)
- net A3: now also M1.4 (B_4)
- net A4: now also M1.5 (B_5)
- net A5: now also M1.6 (B_6)
- net A6: now also M1.7 (B_7)
- net A7: now also M1.8 (B_8)
- net A8: now also M1.9 (R_1)
- net A9: now also M1.10 (R_2)
- net GND: now also R17.1, R18.1, R19.1, R20.1, R21.1, R22.2, R23.2, R24.1, R25.1, R26.1, R27.1
- net RX1/19: now also M1.23 (G_3)
- net RX2/17: now also M1.25 (G_5)
- net RX3/15: now also M1.27 (G_7)
- net SCL/21: now also M1.21 (G_1)
- net SDA/20: now also M1.22 (G_2)
- net TX1/18: now also M1.24 (G_4)
- net TX2/16: now also M1.26 (G_6)
- net TX3/14: now also M1.28 (G_8)
- net at BZ1.2 (+): now also R24.2
- net at M2.20 (P_4): now also R12.2
- net at R25.2: now also BZ2.2 (+)
- net at BZ3.2 (+): now also R26.2
- net at M2.17 (P_1): now also R9.2
- net at M2.18 (P_2): now also R10.2
- net at M2.19 (P_3): now also R11.2
- net at M2.29 (P_5): now also R13.1
- net at M2.30 (P_6): now also R14.1
- net at M2.31 (P_7): now also R15.1
- net at M2.32 (P_8): now also R16.1
- net at M1.32 (P_8): now also R8.1; no longer R5.2
- net at M1.31 (P_7): now also R7.1; no longer R6.2
- net at M1.30 (P_6): now also R6.1; no longer R7.2
- net at BZ4.2 (+): now also R27.2
- net at M1.29 (P_5): now also R5.1; no longer R8.2
- net 1: no longer names the net of M2.1 (B_1)
- net 1: no longer M1.1 (B_1)
- net 10: no longer names the net of M2.10 (R_2)
- net 10: no longer M1.10 (R_2)
- net 11: no longer names the net of M2.11 (R_3)
- net 11: no longer M1.11 (R_3)
- net 12: no longer names the net of M2.12 (R_4)
- net 12: no longer M1.12 (R_4)
- net 13: no longer names the net of M2.13 (R_5)
- net 13: no longer M1.13 (R_5)
- net 14: no longer names the net of M2.14 (R_6)
- net 14: no longer M1.14 (R_6)
- net 15: no longer names the net of M2.15 (R_7)
- net 15: no longer M1.15 (R_7)
- net 16: no longer names the net of M2.16 (R_8)
- net 16: no longer M1.16 (R_8)
- net 2: no longer names the net of M2.2 (B_2)
- net 2: no longer M1.2 (B_2)
- removed net 21: M1.21 (G_1), M2.21 (G_1)
- net 3: no longer names the net of M2.3 (B_3)
- net 3: no longer M1.3 (B_3)
- net 4: no longer names the net of M2.4 (B_4)
- net 4: no longer M1.4 (B_4)
- net 5: no longer names the net of M2.5 (B_5)
- net 5: no longer M1.5 (B_5)
- net 6: no longer names the net of M2.6 (B_6)
- net 6: no longer M1.6 (B_6)
- net 7: no longer names the net of M2.7 (B_7)
- net 7: no longer M1.7 (B_7)
- net 8: no longer names the net of M2.8 (B_8)
- net 8: no longer M1.8 (B_8)
- net 9: no longer names the net of M2.9 (R_1)
- net 9: no longer M1.9 (R_1)
Other:
- moved on the sheet: BZ1, BZ2, BZ3, BZ4, J2, J3, J4, J5, J6, J7, M1, R1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
