File: PCB/Tetris/Tetris.kicad_sch (KiCad schematic)
At the start: 49 parts, among them J1 Power, J2 PWM, J3 Analog, J4 PWM, J5 Analog, J6 Communication, J7 Digital, M1 RGBMatrix, M2 RGBMatrix, SW1 SW_Push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

Commit message: Sync Changes
Connections:
- net *44: now also U1.14 (SER)
- net *46: now also U2.11 (SRCLK); no longer U1.12 (RCLK), U2.12 (RCLK)
- net 22: now also R12.1, R4.1
- net 24: now also R11.1, R3.1
- net 26: now also R10.1, R2.1
- net 28: now also R1.1, R9.1; no longer R12.1, R4.1
- net 30: now also R13.2, R5.2; no longer R11.1, R3.1
- net 32: now also R14.2, R6.2; no longer R10.1, R2.1
- net 34: now also R15.2, R7.2; no longer R1.1, R9.1
- net 36: now also R16.2, R8.2; no longer R13.2, R5.2
- net 38: no longer R14.2, R6.2
- net 40: now also U1.12 (RCLK); no longer R15.2, R7.2
- net 42: now also U1.11 (SRCLK); no longer R16.2, R8.2
- net 48: now also U2.12 (RCLK); no longer U1.11 (SRCLK), U2.11 (SRCLK)
- net 50: now also U2.14 (SER); no longer U1.14 (SER)
- net at U1.9 (QH'): no longer U2.14 (SER)

Commit message: snyc
Connections:
- net 22: no longer R12.1, R4.1
- net 24: now also R12.1, R4.1; no longer R11.1, R3.1
- net 26: now also R11.1, R3.1; no longer R10.1, R2.1
- net 28: now also R10.1, R2.1; no longer R1.1, R9.1
- net 30: now also R1.1, R9.1; no longer R13.2, R5.2
- net 32: now also R13.2, R5.2; no longer R14.2, R6.2
- net 34: now also R14.2, R6.2; no longer R15.2, R7.2
- net 36: now also R15.2, R7.2; no longer R16.2, R8.2
- net 38: now also R16.2, R8.2
Changed lines of the file:
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@@
     (stroke (width 0) (type default))
   )
-  (bus_entry (at 170.18 146.05) (size -2.54 2.54)
+  (bus_entry (at 149.86 146.05) (size -2.54 2.54)
     (stroke (width 0) (type default))
   )
@@
     (stroke (width 0) (type default))
   )
-  (bus (pts (xy 167.64 146.05) (xy 170.18 146.05))
-    (stroke (width 0) (type default))
-  )
   (wire (pts (xy 27.305 44.45) (xy 27.305 29.21))
     (stroke (width 0) (type solid))
@@
     (stroke (width 0) (type default))
   )
+  (bus (pts (xy 149.86 146.05) (xy 152.4 146.05))
+    (stroke (width 0) (type default))
+  )
   (bus (pts (xy 177.8 62.23) (xy 177.8 64.77))
     (stroke (width 0) (type default))
@@
     (stroke (width 0) (type solid))
   )
-  (bus (pts (xy 170.18 146.05) (xy 172.085 146.05))
+  (bus (pts (xy 167.64 146.05) (xy 172.085 146.05))
     (stroke (width 0) (type default))
   )
@@
     (effects (font (size 1.27 1.27)) (justify right bottom))
   )
+  (label "26" (at 169.545 72.39 180) (fields_autoplaced)
+    (effects (font (size 1.27 1.27)) (justify right bottom))
+  )
   (label "31" (at 157.48 181.61 90) (fields_autoplaced)
     (effects (font (size 1.27 1.27)) (justify left bottom))
@@
     (effects (font (size 1.27 1.27)) (justify left bottom))
   )
-  (label "36" (at 168.91 95.25 180) (fields_autoplaced)
+  (label "28" (at 169.545 74.93 180) (fields_autoplaced)
+    (effects (font (size 1.27 1.27)) (justify right bottom))
+  )
+  (label "38" (at 168.91 95.25 180) (fields_autoplaced)
     (effects (font (size 1.27 1.27)) (justify right bottom))
   )
@@
     (effects (font (size 1.27 1.27)) (justify right bottom))
   )
-  (label "28" (at 169.545 133.35 180) (fields_autoplaced)
+  (label "30" (at 169.545 133.35 180) (fields_autoplaced)
+    (effects (font (size 1.27 1.27)) (justify right bottom))
+  )
+  (label "36" (at 169.545 41.91 180) (fields_autoplaced)
     (effects (font (size 1.27 1.27)) (justify right bottom))
   )
@@
     (effects (font (size 1.27 1.27)) (justify left bottom))
   )
-  (label "32" (at 168.91 100.33 180) (fields_autoplaced)
+  (label "34" (at 168.91 100.33 180) (fields_autoplaced)
     (effects (font (size 1.27 1.27)) (justify right bottom))
   )
@@
     (effects (font (size 1.27 1.27)) (justify left bottom))
   )
-  (label "26" (at 169.545 74.93 180) (fields_autoplaced)
-    (effects (font (size 1.27 1.27)) (justify right bottom))
-  )
   (label "S3" (at 119.38 44.45 0) (fields_autoplaced)
     (effects (font (size 1.27 1.27)) (justify left bottom))
@@
     (effects (font (size 1.27 1.27)) (justify left bottom))
   )
+  (label "38" (at 169.545 39.37 180) (fields_autoplaced)
+    (effects (font (size 1.27 1.27)) (justify right bottom))
+  )
   (label "41" (at 144.78 181.61 90) (fields_autoplaced)
     (effects (font (size 1.27 1.27)) (justify left bottom))
   )
-  (label "22" (at 169.545 69.85 180) (fields_autoplaced)
-    (effects (font (size 1.27 1.27)) (justify right bottom))
-  )
   (label "30" (at 157.48 148.59 270) (fields_autoplaced)
     (effects (font (size 1.27 1.27)) (justify right bottom))
@@
     (effects (font (size 1.27 1.27)) (justify right bottom))
   )
-  (label "22" (at 169.545 125.73 180) (fields_autoplaced)
+  (label "24" (at 169.545 125.73 180) (fields_autoplaced)
     (effects (font (size 1.27 1.27)) (justify right bottom))
   )
@@
     (effects (font (size 1.27 1.27)) (justify left bottom))
   )
-  (label "26" (at 169.545 130.81 180) (fields_autoplaced)
+  (label "28" (at 169.545 130.81 180) (fields_autoplaced)
     (effects (font (size 1.27 1.27)) (justify right bottom))
   )
@@
     (effects (font (size 1.27 1.27)) (justify left bottom))
   )
-  (label "30" (at 169.545 46.99 180) (fields_autoplaced)
+  (label "32" (at 169.545 46.99 180) (fields_autoplaced)
     (effects (font (size 1.27 1.27)) (justify right bottom))
   )
@@
     (effects (font (size 1.27 1.27)) (justify right bottom))
   )
-  (label "28" (at 169.545 77.47 180) (fields_autoplaced)
-    (effects (font (size 1.27 1.27)) (justify right bottom))
-  )
   (label "*9" (at 175.26 67.31 180) (fields_autoplaced)
     (effects (font (size 1.27 1.27)) (justify right bottom))
@@
     (effects (font (size 1.27 1.27)) (justify right bottom))
   )
-  (label "30" (at 168.91 102.87 180) (fields_autoplaced)
+  (label "32" (at 168.91 102.87 180) (fields_autoplaced)
     (effects (font (size 1.27 1.27)) (justify right bottom))
   )
@@
     (effects (font (size 1.27 1.27)) (justify left bottom))
   )
-  (label "24" (at 169.545 72.39 180) (fields_autoplaced)
-    (effects (font (size 1.27 1.27)) (justify right bottom))
-  )
   (label "*3" (at 202.565 100.33 0) (fields_autoplaced)
     (effects (font (size 1.27 1.27)) (justify left bottom))
   )
-  (label "34" (at 168.91 97.79 180) (fields_autoplaced)
-    (effects (font (size 1.27 1.27)) (justify right bottom))
-  )
-  (label "32" (at 169.545 44.45 180) (fields_autoplaced)
+  (label "36" (at 168.91 97.79 180) (fields_autoplaced)
     (effects (font (size 1.27 1.27)) (justify right bottom))
   )
@@
     (effects (font (size 1.27 1.27)) (justify right bottom))
   )
+  (label "34" (at 169.545 44.45 180) (fields_autoplaced)
+    (effects (font (size 1.27 1.27)) (justify right bottom))
+  )
   (label "AREF" (at 202.565 65.405 0) (fields_autoplaced)
     (effects (font (size 1.27 1.27)) (justify left bottom))
@@
     (effects (font (size 1.27 1.27)) (justify right bottom))
   )
-  (label "24" (at 169.545 128.27 180) (fields_autoplaced)
+  (label "26" (at 169.545 128.27 180) (fields_autoplaced)
     (effects (font (size 1.27 1.27)) (justify right bottom))
   )
@@
     (effects (font (size 1.27 1.27)) (justify right bottom))
   )
+  (label "24" (at 169.545 69.85 180) (fields_autoplaced)
+    (effects (font (size 1.27 1.27)) (justify right bottom))
+  )
   (label "27" (at 162.56 181.61 90) (fields_autoplaced)
     (effects (font (size 1.27 1.27)) (justify left bottom))
@@
     (effects (font (size 1.27 1.27)) (justify left bottom))
   )
-  (label "34" (at 169.545 41.91 180) (fields_autoplaced)
-    (effects (font (size 1.27 1.27)) (justify right bottom))
-  )
   (label "*6" (at 202.565 92.71 0) (fields_autoplaced)
     (effects (font (size 1.27 1.27)) (justify left bottom))
@@
     (effects (font (size 1.27 1.27)) (justify left bottom))
   )
+  (label "30" (at 169.545 77.47 180) (fields_autoplaced)
+    (effects (font (size 1.27 1.27)) (justify right bottom))
+  )
   (label "A7" (at 36.83 107.95 180) (fields_autoplaced)
     (effects (font (size 1.27 1.27)) (justify right bottom))
   )
-  (label "36" (at 169.545 39.37 180) (fields_autoplaced)
-    (effects (font (size 1.27 1.27)) (justify right bottom))
-  )
