File: PCB/Tetris/Tetris_Copy_3.kicad_pcb (KiCad board)
At the start: 2 copper layers, 49 parts, among them J1 Power, J2 PWM, J3 Analog, J4 PWM, J5 Analog, J6 Communication, J7 Digital, M1 RGBMatrix, M2 RGBMatrix, SW1 SW_Push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

Commit message: Saving progress
Parts:
- removed U2: 74HC595, Package_DIP:DIP-16_W7.62mm_Socket_LongPads
- J1: footprint Connector_PinHeader_2.54mm:PinHeader_1x08_P2.54mm_Vertical -> Connector_PinSocket_2.54mm:PinSocket_1x08_P2.54mm_Vertical; moved to F.Cu
- moved U1 52.9 mm to (151.5, 111.9), turned to -90 degrees
- moved R3 4.35 mm to (174.7, 104.0)
- moved R1 4.35 mm to (180.9, 104.0)
- moved R2 4.35 mm to (177.8, 104.0)
- moved R4 4.35 mm to (171.6, 104.0)
- moved R10 3.15 mm to (136.5, 102.2)
- moved R12 3.10 mm to (130.3, 102.2)
- moved R11 3.08 mm to (127.2, 102.2)
- moved R9 3.03 mm to (133.4, 102.2)
- turned J1 to 90 degrees
Connections:
- M2 pad 1: /S1 -> unconnected-(M2-B_1-Pad1)
- M2 pad 10: /S10 -> unconnected-(M2-R_2-Pad10)
- M2 pad 11: /S11 -> unconnected-(M2-R_3-Pad11)
- M2 pad 12: /S12 -> unconnected-(M2-R_4-Pad12)
- M2 pad 13: /S13 -> unconnected-(M2-R_5-Pad13)
- M2 pad 14: /S14 -> unconnected-(M2-R_6-Pad14)
- M2 pad 15: /S15 -> unconnected-(M2-R_7-Pad15)
- M2 pad 16: /S16 -> unconnected-(M2-R_8-Pad16)
- M2 pad 2: /S2 -> unconnected-(M2-B_2-Pad2)
- M2 pad 3: /S3 -> unconnected-(M2-B_3-Pad3)
- M2 pad 4: /S4 -> unconnected-(M2-B_4-Pad4)
- M2 pad 5: /S5 -> unconnected-(M2-B_5-Pad5)
- M2 pad 6: /S6 -> unconnected-(M2-B_6-Pad6)
- M2 pad 7: /S7 -> unconnected-(M2-B_7-Pad7)
- M2 pad 8: /S8 -> unconnected-(M2-B_8-Pad8)
- M2 pad 9: /S9 -> unconnected-(M2-R_1-Pad9)
- R1 pad 1: /34 -> /A
- R10 pad 1: /32 -> /B
- R11 pad 1: /30 -> /C
- R12 pad 1: /28 -> /D
- R13 pad 2: /36 -> /E
- R14 pad 2: /38 -> /F
- R15 pad 2: /40 -> /G
- R16 pad 2: /42 -> /H
- R2 pad 1: /32 -> /B
- R3 pad 1: /30 -> /C
- R4 pad 1: /28 -> /D
- R5 pad 2: /36 -> /E
- R6 pad 2: /38 -> /F
- R7 pad 2: /40 -> /G
- R8 pad 2: /42 -> /H
- R9 pad 1: /34 -> /A
- U1 pad 1: /S2 -> /B
- U1 pad 11: /48 -> /49
- U1 pad 12: /*46 -> /51
- U1 pad 14: /50 -> /53
- U1 pad 15: /S1 -> /A
- U1 pad 2: /S3 -> /C
- U1 pad 3: /S4 -> /D
- U1 pad 4: /S5 -> /E
- U1 pad 5: /S6 -> /F
- U1 pad 6: /S7 -> /G
- U1 pad 7: /S8 -> /H
- U1 pad 9: Net-(U1-QH') -> unconnected-(U1-QH'-Pad9)
Routing:
- net /A: track 0.00 -> 95.0 mm
- net /50: track 88.4 -> 0.00 mm
- net /49: track 0.00 -> 88.0 mm
- net /*46: track 86.0 -> 0.00 mm
- net /48: track 85.1 -> 0.00 mm
- net /B: track 0.00 -> 85.0 mm
- net /51: track 0.00 -> 69.2 mm
- net /53: track 0.00 -> 61.3 mm
- net /32: track 59.7 -> 0.00 mm
- net /34: track 55.9 -> 0.00 mm
- net /42: track 45.9 -> 0.00 mm
- net /40: track 42.6 -> 0.00 mm
- net +5V: track 151.5 -> 112.1 mm
- net /38: track 39.3 -> 0.00 mm
- net /36: track 36.0 -> 0.00 mm
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