File: PCB/Tetris/_autosave-Tetris.kicad_sch (KiCad schematic)
At the start: 49 parts, among them J1 Power, J2 PWM, J3 Analog, J4 PWM, J5 Analog, J6 Communication, J7 Digital, M1 RGBMatrix, M2 RGBMatrix, SW1 SW_Push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

Commit message: Saving progress
Changed lines of the file:
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@@
+    (stroke (width 0) (type default))
+  )
+  (bus_entry (at 116.84 44.45) (size 2.54 2.54)
     (stroke (width 0) (type default))
   )
@@
     (stroke (width 0) (type default))
   )
+  (bus_entry (at 33.655 43.815) (size 2.54 -2.54)
+    (stroke (width 0) (type default))
+  )
   (bus_entry (at 175.26 52.07) (size 2.54 -2.54)
     (stroke (width 0) (type default))
@@
     (stroke (width 0) (type default))
   )
-  (bus_entry (at 119.38 46.99) (size -2.54 -2.54)
-    (stroke (width 0) (type default))
-  )
   (bus_entry (at 169.545 125.73) (size 2.54 2.54)
     (stroke (width 0) (type default))
@@
     (stroke (width 0) (type default))
   )
-  (bus_entry (at 33.655 43.815) (size 2.54 -2.54)
-    (stroke (width 0) (type default))
-  )
